File: Maestro Mini/Maestro Mini.kicad_pcb (KiCad board)
At the start: 2 copper layers, 22 parts, among them J1 Conn_01x03, SW1 SW_Push, SW10 SW_Push, SW11 SW_SPDT, SW2 SW_Push, SW3 SW_Push, SW4 SW_Push, SW5 SW_Push, SW6 SW_Push, SW7 SW_Push, SW8 SW_Push, SW9 SW_Push, U1 MCP23017x-x-SP, U2 XIAO-ESP32-C3-SMD

Commit message: Finalized PCB design and updated schematics.
Parts:
- removed BT1: Battery_Cell, Connector_PinHeader_2.54mm:PinHeader_1x02_P2.54mm_Vertical
- removed J1: Conn_01x03, Connector_PinHeader_2.54mm:PinHeader_1x03_P2.54mm_Vertical
- removed LS1: Speaker, Connector_PinHeader_2.54mm:PinHeader_1x02_P2.54mm_Vertical
- removed SW11: SW_SPDT, Connector_PinHeader_2.54mm:PinHeader_1x03_P2.54mm_Vertical
- SW1, SW10, SW2, SW3, SW4, SW5, SW6, SW7, SW8, SW9: footprint Button_Switch_Keyboard:SW_Cherry_MX_1.00u_PCB -> Imported Parts:Test_SW_Cherry_MX_1.00u_PCB
- moved OLED1 91.6 mm to (175.3, 42.6)
- moved AdafruitPAM8302 80.0 mm to (133.3, 59.5)
- moved SW1 80.0 mm to (118.3, 124.5)
- moved SW2 80.0 mm to (118.3, 102.5)
- moved SW3 80.0 mm to (118.5, 80.6)
- moved SW4 80.0 mm to (118.3, 58.5)
- moved SW5 80.0 mm to (140.5, 124.6)
- moved SW6 80.0 mm to (140.3, 102.5)
- moved SW7 80.0 mm to (140.3, 80.5)
- moved U2 80.0 mm to (168.6, 118.4)
- moved U1 77.8 mm to (167.5, 79.6)
- moved R1 77.3 mm to (153.3, 95.6)
- moved R2 77.3 mm to (153.3, 90.1)
- moved SW10 74.5 mm to (191.8, 80.0)
- moved SW8 74.5 mm to (191.8, 124.0)
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Connections:
- U2 pad 21: Net-(SW11-B) -> unconnected-(U2-VBAT-Pad21)
Routing:
- net +3V3: track 0.00 -> 201.2 mm, vias 0 -> 3
- net /SCL: track 0.00 -> 140.8 mm
- net /SDA: track 0.00 -> 114.2 mm
- net /BTN_F: track 0.00 -> 105.3 mm
- net /BTN_E: track 0.00 -> 104.3 mm
- net /BTN_D: track 0.00 -> 86.5 mm
- net /BTN_FL: track 0.00 -> 84.3 mm
- net /BTN_C: track 0.00 -> 74.0 mm
- net Net-(AdafruitPAM8302-Pin_1): track 0.00 -> 61.5 mm
- net /BTN_SH: track 0.00 -> 56.2 mm
- net /BTN_G: track 0.00 -> 52.7 mm
- net /BTN_A: track 0.00 -> 42.2 mm
- net /BTN_B: track 0.00 -> 39.9 mm
- net /BTN_CTRL: track 0.00 -> 27.5 mm
- net /AUDIO_OUT: track 0.00 -> 25.3 mm
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- added copper zone on B.Cu, net GND
- added copper zone on F.Cu, net GND
Other:
- board outline added: 104.9 x 110 mm
